Commit message: Gazebo update 1

File: description/robot.urdf.xacro (robot description, xacro)
@@ -4,3 +4,4 @@
     <!-- <link name="base_link"></link> -->
     <xacro:include filename="robot_core.xacro"/>
+    <xacro:include filename="gazebo_control.xacro"/>
 </robot>

File: description/robot_core.xacro (robot description, xacro)
@@ -41,4 +41,7 @@
         </xacro:inertial_box>
     </link>
+    <gazebo reference="chassis_link">
+        <material>Gazebo/White</material>
+    </gazebo>
     <!-- Left wheel -->
     <joint name="left_wheel_joint" type="continuous">
@@ -65,4 +68,7 @@
         </xacro:inertial_cylinder>
     </link>
+    <gazebo reference="left_wheel_link">
+        <material>Gazebo/Blue</material>
+    </gazebo>
     <!-- Right wheel -->
     <joint name="right_wheel_joint" type="continuous">
@@ -71,5 +77,5 @@
         <child link="right_wheel_link"/>
         <origin xyz="0.0 -0.175 0.0" rpy="${pi/2} 0.0 0.0"/>
-        <axis xyz="0.0 0.0 1.0"/>
+        <axis xyz="0.0 0.0 -1.0"/>
     </joint>
     <link name="right_wheel_link">
@@ -89,4 +95,7 @@
         </xacro:inertial_cylinder>
     </link>
+    <gazebo reference="right_wheel_link">
+        <material>Gazebo/Blue</material>
+    </gazebo>
     <!-- Caster wheel -->
     <joint name="caster_joint" type="fixed">
@@ -111,3 +120,8 @@
         </xacro:inertial_sphere>
     </link>
+    <gazebo reference="caster_wheel_link">
+        <material>Gazebo/Black</material>
+        <mu1 value="0.001"/>
+        <mu2 value="0.001"/>
+    </gazebo>
 </robot>

Commit message: Final simu robot model

File: description/robot.urdf.xacro (robot description, xacro)
@@ -3,5 +3,9 @@
     <!-- Example link -->
     <!-- <link name="base_link"></link> -->
+    <!-- Descript main robot -->
     <xacro:include filename="robot_core.xacro"/>
+    <!-- For Gazebo simulation -->
     <xacro:include filename="gazebo_control.xacro"/>
+    <!-- Lidar -->
+    <xacro:include filename="lidar.xacro"/>
 </robot>

File: description/robot_core.xacro (robot description, xacro)
@@ -14,4 +14,7 @@
     <material name="black">
         <color rgba="0.0 0.0 0.0 1.0"/>
+    </material>
+    <material name="red">
+        <color rgba="1.0 0.0 0.0 1.0"/>
     </material>
     <!-- Base -->
