Commit message: change name: lidar -> laser

File: description/lidar.xacro (robot description, xacro)
@@ -3,8 +3,8 @@
     <joint name="lidar_joint" type="fixed">
         <parent link="chassis_link"/>
-        <child link="lidar_link"/>
+        <child link="laser_frame"/>
         <origin xyz="0.1 0.0 0.175" rpy="0.0 0.0 0.0"/>
     </joint>
-    <link name="lidar_link">
+    <link name="laser_frame">
         <visual>
             <geometry>
@@ -22,8 +22,8 @@
         </xacro:inertial_cylinder>
     </link>
-    <gazebo reference="lidar_link">
+    <gazebo reference="laser_frame">
         <material>Gazebo/Red</material>
         <!-- The name of sensor is not fixed -->
-        <sensor name="lidar" type="ray">
+        <sensor name="laser" type="ray">
             <!-- The same origin with the link -->
             <pose> 0 0 0 0 0 0 </pose>
@@ -44,5 +44,5 @@
             </ray>
             <!-- The name does not matter -->
-            <plugin name="Lidar_controller" filename="libgazebo_ros_ray_sensor.so">
+            <plugin name="laser_controller" filename="libgazebo_ros_ray_sensor.so">
                 <!-- What topic to publish -->
                 <ros>
@@ -50,5 +50,5 @@
                 </ros>
                 <output_type>sensor_msgs/LaserScan</output_type>
-                <frame_name>lidar_link</frame_name>
+                <frame_name>laser_frame</frame_name>
             </plugin>
         </sensor>
