Commit message: Add new robot model

File: description/model_2/ego_racecar.xacro (robot description, xacro)
@@ -12,15 +12,29 @@
   <xacro:property name="laser_radius" value="0.026" />
   <xacro:property name="car_name" value="ego_racecar" />
+  <xacro:include filename="inertial_macros.xacro"/>
+  <!-- For Gazebo simulation -->
+  <xacro:include filename="gazebo_control.xacro"/>
+  <!-- Lidar -->
+  <xacro:include filename="lidar.xacro"/>
   <!-- Colors -->
-  <material name="black">
-    <color rgba="0.2 0.2 0.2 1."/>
+  <material name="white">
+    <color rgba="1.0 1.0 1.0 1.0"/>
+  </material>
+  <material name="orange">
+    <color rgba="1.0 0.3 0.1 1.0"/>
   </material>
   <material name="blue">
-    <color rgba="0.3 0.57 1. 1."/>
+    <color rgba="0.2 0.2 1.0 1.0"/>
+  </material>
+  <material name="black">
+    <color rgba="0.0 0.0 0.0 1.0"/>
+  </material>
+  <material name="red">
+    <color rgba="1.0 0.0 0.0 1.0"/>
   </material>
   <!-- Base link -->
   <link name="${car_name}/base_link">
     <visual>
-      <origin xyz="${wheelbase/2} 0 ${ground_offset+height/2}"/>
+      <origin xyz="${wheelbase/2} 0.0 ${ground_offset+height/2}"/>
       <geometry>
         <box size="${wheelbase} ${width} ${height}"/>
@@ -28,21 +42,19 @@
       <material name="blue"/>
     </visual>
+    <collision>
+      <origin xyz="${wheelbase/2} 0 ${ground_offset+height/2}"/>
+      <geometry>
+        <box size="${wheelbase} ${width} ${height}"/>
+      </geometry>
+    </collision>
+    <xacro:inertial_box mass="0.5" x="${wheelbase}" y="${width}" z="${height}">
+      <origin xyz="${wheelbase/2} 0.0 ${ground_offset+height/2}" rpy="0.0 0.0 0.0"/>
+    </xacro:inertial_box>
   </link>
-  <!-- Laser -->
-  <joint name="base_to_laser_model" type="fixed">
-    <parent link="${car_name}/base_link"/>
-    <child link="${car_name}/laser_model"/>
-    <origin xyz="${laser_distance_from_base_link} 0 ${ground_offset+height+(laser_height/2)}"/>
-  </joint>
-  <link name="${car_name}/laser_model">
-    <visual>
-      <geometry>
-        <cylinder radius="${laser_radius}" length="${laser_height}"/>
-      </geometry>
-      <material name="black"/>
-    </visual>
-  </link>
+  <gazebo reference="${car_name}/base_link">
+    <material>Gazebo/Blue</material>
+  </gazebo>
   <!-- Back left wheel -->
-  <joint name="$base_to_back_left_wheel" type="continuous">
+  <joint name="base_to_back_left_wheel" type="continuous">
     <parent link="${car_name}/base_link"/>
     <child link="${car_name}/back_left_wheel"/>
@@ -56,7 +68,17 @@
       </geometry>
       <material name="black"/>
-      <!-- <origin rpy="$-{pi/2} 0.0 0.0"/> -->
     </visual>
+    <collision>
+      <geometry>
+        <cylinder radius="${wheel_radius}" length="${wheel_length}"/>
+      </geometry>
+    </collision>
+    <xacro:inertial_cylinder mass="0.1" length="${wheel_length}" radius="${wheel_radius}">
+      <origin xyz="0.0 0.0 0.0" rpy="0.0 0.0 0.0"/>
+    </xacro:inertial_cylinder>
   </link>
+  <gazebo reference="${car_name}/back_left_wheel">
+    <material>Gazebo/Black</material>
+  </gazebo>
   <!-- Back right wheel -->
   <joint name="base_to_back_right_wheel" type="continuous">
@@ -72,9 +94,19 @@
       </geometry>
       <material name="black"/>
-      <!-- <origin rpy="${pi/2} 0.0 0.0"/> -->
     </visual>
+    <collision>
+      <geometry>
+        <cylinder radius="${wheel_radius}" length="${wheel_length}"/>
+      </geometry>
+    </collision>
+    <xacro:inertial_cylinder mass="0.1" length="${wheel_length}" radius="${wheel_radius}">
+      <origin xyz="0.0 0.0 0.0" rpy="0.0 0.0 0.0"/>
+    </xacro:inertial_cylinder>
   </link>
+  <gazebo reference="${car_name}/back_right_wheel">
+    <material>Gazebo/Black</material>
+  </gazebo>
   <!-- Front left wheel & hinge -->
-  <!-- B2F LH -->
+  <!-- Left hinge [Joint] -->
   <joint name="base_to_front_left_hinge" type="fixed">
     <parent link="${car_name}/base_link"/>
@@ -82,7 +114,7 @@
     <origin xyz="${wheelbase} ${(wheel_length+width)/2} ${wheel_radius}" rpy="-${pi/2} 0.0 0.0"/>
   </joint>
-  <!-- F LH -->
+  <!-- Left hinge [Link] -->
   <link name="${car_name}/front_left_hinge"/>
-  <!-- F LH2W -->
+  <!-- Front left wheel [Joint] -->
   <joint name="front_left_hinge_to_wheel" type="continuous">
     <parent link="${car_name}/front_left_hinge"/>
@@ -91,5 +123,5 @@
     <axis xyz="0.0 0.0 1.0"/>
   </joint>
-  <!-- F LW -->
+  <!-- Front left wheel [Link] -->
   <link name="${car_name}/front_left_wheel">
     <visual>
@@ -98,9 +130,19 @@
       </geometry>
       <material name="black"/>
-      <!-- <origin xyz="0.0 0.0 0.0" rpy="$-{pi/2} 0.0 0.0"/> -->
     </visual>
+    <collision>
+      <geometry>
+        <cylinder radius="${wheel_radius}" length="${wheel_length}"/>
+      </geometry>
+    </collision>
+    <xacro:inertial_cylinder mass="0.1" length="${wheel_length}" radius="${wheel_radius}">
+      <origin xyz="0.0 0.0 0.0" rpy="0.0 0.0 0.0"/>
+    </xacro:inertial_cylinder>
   </link>
+  <gazebo reference="${car_name}/front_left_wheel">
+    <material>Gazebo/Black</material>
+  </gazebo>
   <!-- Front right wheel & hinge -->
-  <!-- B2F RH -->
+  <!-- Right hinge [Joint] -->
   <joint name="base_to_front_right_hinge" type="fixed">
     <parent link="${car_name}/base_link"/>
@@ -108,7 +150,7 @@
     <origin xyz="${wheelbase} ${-(wheel_length+width)/2} ${wheel_radius}" rpy="${pi/2} 0.0 0.0"/>
   </joint>
-  <!-- F RH -->
+  <!-- Right hinge [Link] -->
   <link name="${car_name}/front_right_hinge"/>
-  <!-- F RH2W -->
+  <!-- Front right wheel [Joint] -->
   <joint name="front_right_hinge_to_wheel" type="continuous">
     <parent link="${car_name}/front_right_hinge"/>
@@ -117,5 +159,5 @@
     <axis xyz="0.0 0.0 -1.0"/>
   </joint>
-  <!-- F RW -->
+  <!-- Front right wheel [Link] -->
   <link name="${car_name}/front_right_wheel">
     <visual>
@@ -124,6 +166,16 @@
       </geometry>
       <material name="black"/>
-      <!-- <origin xyz="0.0 0.0 0.0" rpy="${pi/2} 0.0 0.0"/> -->
     </visual>
+    <collision>
+      <geometry>
+        <cylinder radius="${wheel_radius}" length="${wheel_length}"/>
+      </geometry>
+    </collision>
+    <xacro:inertial_cylinder mass="0.1" length="${wheel_length}" radius="${wheel_radius}">
+      <origin xyz="0.0 0.0 0.0" rpy="0.0 0.0 0.0"/>
+    </xacro:inertial_cylinder>
   </link>
+  <gazebo reference="${car_name}/front_right_wheel">
+    <material>Gazebo/Black</material>
+  </gazebo>
 </robot>

Commit message: Fixed back wheels

File: description/model_2/ego_racecar.xacro (robot description, xacro)
@@ -56,5 +56,5 @@
   </gazebo>
   <!-- Back left wheel -->
-  <joint name="base_to_back_left_wheel" type="continuous">
+  <joint name="base_to_back_left_wheel" type="fixed">
     <parent link="${car_name}/base_link"/>
     <child link="${car_name}/back_left_wheel"/>
@@ -82,5 +82,5 @@
   </gazebo>
   <!-- Back right wheel -->
-  <joint name="base_to_back_right_wheel" type="continuous">
+  <joint name="base_to_back_right_wheel" type="fixed">
     <parent link="${car_name}/base_link"/>
     <child link="${car_name}/back_right_wheel"/>

Commit message: Fixed front wheel & move back wheel

File: description/model_2/ego_racecar.xacro (robot description, xacro)
@@ -56,5 +56,5 @@
   </gazebo>
   <!-- Back left wheel -->
-  <joint name="base_to_back_left_wheel" type="fixed">
+  <joint name="base_to_back_left_wheel" type="continuous">
     <parent link="${car_name}/base_link"/>
     <child link="${car_name}/back_left_wheel"/>
@@ -82,5 +82,5 @@
   </gazebo>
   <!-- Back right wheel -->
-  <joint name="base_to_back_right_wheel" type="fixed">
+  <joint name="base_to_back_right_wheel" type="continuous">
     <parent link="${car_name}/base_link"/>
     <child link="${car_name}/back_right_wheel"/>
@@ -117,5 +117,5 @@
   <link name="${car_name}/front_left_hinge"/>
   <!-- Front left wheel [Joint] -->
-  <joint name="front_left_hinge_to_wheel" type="continuous">
+  <joint name="front_left_hinge_to_wheel" type="fixed">
     <parent link="${car_name}/front_left_hinge"/>
     <child link="${car_name}/front_left_wheel"/>
@@ -153,5 +153,5 @@
   <link name="${car_name}/front_right_hinge"/>
   <!-- Front right wheel [Joint] -->
-  <joint name="front_right_hinge_to_wheel" type="continuous">
+  <joint name="front_right_hinge_to_wheel" type="fixed">
     <parent link="${car_name}/front_right_hinge"/>
     <child link="${car_name}/front_right_wheel"/>
