Commit message: Add base footprint

File: description/model_1/robot_core.xacro (robot description, xacro)
@@ -20,4 +20,11 @@
     <!-- Base -->
     <link name="base_link"/>
+    <!-- Base footprint -->
+    <joint name="base_footprint_joint" type="fixed">
+        <parent link="base_link"/>
+        <child link="base_footprint"/>
+        <origin xyz="0 0 0" rpy="0 0 0"/>
+    </joint>
+    <link name="base_footprint"></link>
     <!-- Chassis -->
     <joint name="chassis_joint" type="fixed">
