Commit message: laser_frame -> laser

File: description/model_1/lidar.xacro (robot description, xacro)
@@ -3,8 +3,8 @@
     <joint name="lidar_joint" type="fixed">
         <parent link="chassis_link"/>
-        <child link="laser_frame"/>
+        <child link="laser"/>
         <origin xyz="0.1 0.0 0.175" rpy="0.0 0.0 0.0"/>
     </joint>
-    <link name="laser_frame">
+    <link name="laser">
         <visual>
             <geometry>
@@ -22,5 +22,5 @@
         </xacro:inertial_cylinder>
     </link>
-    <gazebo reference="laser_frame">
+    <gazebo reference="laser">
         <material>Gazebo/Red</material>
         <!-- The name of sensor is not fixed -->
@@ -50,5 +50,5 @@
                 </ros>
                 <output_type>sensor_msgs/LaserScan</output_type>
-                <frame_name>laser_frame</frame_name>
+                <frame_name>laser</frame_name>
             </plugin>
         </sensor>

Commit message: Robot color, visual slam map, lidar

File: description/model_1/lidar.xacro (robot description, xacro)
@@ -11,5 +11,5 @@
                 <cylinder radius="0.05" length="0.04"/>
             </geometry>
-            <material name="red"/>
+            <material name="orage"/>
         </visual>
         <collision>
@@ -23,5 +23,5 @@
     </link>
     <gazebo reference="laser">
-        <material>Gazebo/Red</material>
+        <material>Gazebo/Orange</material>
         <!-- The name of sensor is not fixed -->
         <sensor name="laser" type="ray">

File: description/model_1/robot_core.xacro (robot description, xacro)
@@ -39,5 +39,5 @@
                 <box size="0.3 0.3 0.15"/>
             </geometry>
-            <material name="white"/>
+            <material name="blue"/>
         </visual>
         <collision>
@@ -52,5 +52,5 @@
     </link>
     <gazebo reference="chassis_link">
-        <material>Gazebo/White</material>
+        <material>Gazebo/Blue</material>
     </gazebo>
     <!-- Left wheel -->
@@ -67,5 +67,5 @@
                 <cylinder radius="0.05" length="0.04"/>
             </geometry>
-            <material name="blue"/>
+            <material name="black"/>
         </visual>
         <collision>
@@ -79,5 +79,5 @@
     </link>
     <gazebo reference="left_wheel_link">
-        <material>Gazebo/Blue</material>
+        <material>Gazebo/Black</material>
     </gazebo>
     <!-- Right wheel -->
@@ -94,5 +94,5 @@
                 <cylinder radius="0.05" length="0.04"/>
             </geometry>
-            <material name="blue"/>
+            <material name="black"/>
         </visual>
         <collision>
@@ -106,5 +106,5 @@
     </link>
     <gazebo reference="right_wheel_link">
-        <material>Gazebo/Blue</material>
+        <material>Gazebo/Black</material>
     </gazebo>
     <!-- Caster wheel -->
@@ -119,5 +119,5 @@
                 <sphere radius="0.05"/>
             </geometry>
-            <material name="black"/>
+            <material name="white"/>
         </visual>
         <collision>
@@ -131,5 +131,5 @@
     </link>
     <gazebo reference="caster_wheel_link">
-        <material>Gazebo/Black</material>
+        <material>Gazebo/White</material>
         <mu1 value="0.001"/>
         <mu2 value="0.001"/>

Commit message: Fix color name

File: description/model_1/lidar.xacro (robot description, xacro)
@@ -11,5 +11,5 @@
                 <cylinder radius="0.05" length="0.04"/>
             </geometry>
-            <material name="orage"/>
+            <material name="orange"/>
         </visual>
         <collision>
